File: railclock.kicad_sch (KiCad schematic)
At the start: 177 parts, among them J1 Conn_01x02_Pin, J10 Conn_01x04_MountingPin, J11 Conn_01x04_MountingPin, J12 Conn_01x04_MountingPin, J13 Conn_01x04_MountingPin, J14 Conn_01x04_MountingPin, J15 Conn_01x03_MountingPin, J16 Barrel_Jack_Switch, J2 Conn_01x03_MountingPin, J3 Conn_01x04_MountingPin, J4 USB_C_Receptacle_USB2.0_14P, J5 Conn_01x03_MountingPin, J6 Conn_01x03_MountingPin, J7 Conn_01x03_MountingPin, J8 Conn_01x03_MountingPin, J9 Conn_01x04_MountingPin, Q1 Q_NPN_BEC, SW1 SW_SPST, SW2 SW_DPDT_x2, U1 MCP7940N-xST, U10 74AHC1G04, U11 MAX811TEUS-T, U12 MCP4728, U13 BTS5012SDA, U14 BTS5012SDA, U15 BTS5012SDA, U16 BTS5012SDA, U17 BTS5012SDA, U2 MCP73832-2-OT, U4 ESP32-C6-WROOM-1, U5 DRV8870DDA, U6 PAM2421, U8 BQ24296MRGET, U9 PCF8574RGTR, Y1 MC-306_32.7680K-A5__ROHS

Commit message: Schematic marking updates
Parts:
- BT2, BT3, BT4: value Battery_Cell -> 18650
- C10, C13, C22, C24, C27, C32, C33, C34, C35, C36, C37, C9: value C -> 100nF
- C11, C12, C8: value C_Polarized -> 470uF
- D1: value D -> Duża
- D10, D11, D12, D13, D14, D15, D16, D17, D18, D19, D3, D4, D5, D7, D8, D9: value D_Zener -> TVS
- L2: value L -> 1uH
- R11: value R -> 56k
- R17, R18: now not fitted
- R21, R24, R25, R27, R29, R40, R41, R5, R6, R9: value R -> 10k
- R26: value R -> 47k
- R28: value R -> 130k
- R42, R43: value R -> 100R
- R45, R46, R48, R50, R52, R55: value R -> 0R
- R54: value R -> 0R; now not fitted
- R84: value R -> 220R
- RV1: value R_Potentiometer -> 10k
Other:
- moved on the sheet: BT2, BT3, BT4, C10, C11, C12, C13, C14, C15, C18, C19, C20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

Commit message: more values
Parts:
- C25, C30: value C -> 100nF
- C32: footprint Capacitor_SMD:C_0805_2012Metric -> r12
- U3: value ~ -> MIC2545
- U7: value ~ -> TPS73733DCQR
Changed lines of the file:
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@@
 		(on_board yes)
 		(dnp no)
-		(fields_autoplaced yes)
 		(property "Reference" "U7"
-			(at 200.025 166.3785 0)
+			(at 199.898 165.608 0)
 			(effects
 				(font
@@
 			)
 		)
-		(property "Value" "~"
-			(at 200.025 168.0599 0)
+		(property "Value" "TPS73733DCQR"
+			(at 199.898 167.2894 0)
 			(effects
 				(font
@@
 		(fields_autoplaced yes)
 		(property "Reference" "C25"
-			(at 204.851 24.1878 0)
+			(at 205.74 24.1299 0)
 			(effects
 				(font
@@
 			)
 		)
-		(property "Value" "C"
-			(at 204.851 26.6121 0)
+		(property "Value" "100nF"
+			(at 205.74 26.6699 0)
 			(effects
 				(font
@@
 		(fields_autoplaced yes)
 		(property "Reference" "C30"
-			(at 213.741 332.7978 0)
+			(at 214.63 332.7399 0)
 			(effects
 				(font
@@
 			)
 		)
-		(property "Value" "C"
-			(at 213.741 335.2221 0)
+		(property "Value" "100nF"
+			(at 214.63 335.2799 0)
 			(effects
 				(font
@@
 			)
 		)
-		(property "Value" "~"
+		(property "Value" "MIC2545"
 			(at 270.51 293.6629 0)
 			(effects
@@
 			)
 		)
-		(property "Footprint" "Capacitor_SMD:C_0805_2012Metric"
+		(property "Footprint" "r12"
 			(at 227.0252 313.69 0)
 			(effects
